File: hardware/AnalogInBuffers.sch (KiCad schematic (older format))
At the start: 13 parts, among them U11 MCP6004

Commit message: Finish up first plausible version
Parts:
- added C18, C19, C20: 0.1uF, Capacitor_SMD:C_0603_1608Metric_Pad1.08x0.95mm_HandSolder, symbol Device:C_Small
- added C21, C22, C23, C24, C25, C26, C27, C28, C29, C30, C31, C32: 22pF, Capacitor_SMD:C_0603_1608Metric_Pad1.08x0.95mm_HandSolder, symbol Device:C_Small
- added R35, R37, R39, R41, R47, R49, R51, R53: 100k, Resistor_SMD:R_0603_1608Metric_Pad0.98x0.95mm_HandSolder, symbol Device:R_US
- added R36, R38, R40, R42, R48, R50, R52, R54: 121k, Resistor_SMD:R_0603_1608Metric_Pad0.98x0.95mm_HandSolder, symbol Device:R_US
- added R43, R44, R45, R46, R55, R56, R57, R58: 18.7k, Resistor_SMD:R_0603_1608Metric_Pad0.98x0.95mm_HandSolder, symbol Device:R_US
- added unit 5 of U11
- added U12, U13: MCP6004, Package_SO:TSSOP-14_4.4x5mm_P0.65mm, symbol winterbloom:MCP6004
- R23, R24, R25, R26, R27, R28, R29, R30, R31, R32, R33, R34: footprint Resistor_SMD:R_0603_1608Metric_Pad1.05x0.95mm_HandSolder -> Resistor_SMD:R_0603_1608Metric_Pad0.98x0.95mm_HandSolder
Connections:
- net -10V: now also R36.2, R38.2, R40.2, R42.2, R48.2, R50.2, R52.2, R54.2
- net at R23.1, R24.1, R31.2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: now also C21.1
- net GND: now reaches U11.3 (+)
- net GND: now also U11.10 (+), U11.12 (+), U11.5 (+), C18.2, C19.2, C20.2, U11.11 (V-), U12.10 (+), U12.11 (V-), U12.12 (+), U12.3 (+), U12.5 (+), U13.10 (+), U13.11 (V-), U13.12 (+), U13.3 (+), U13.5 (+)
- net at R25.1, R26.1, R32.2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: now also C22.1
- net at R27.1, R28.1, R33.2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: now also C23.1
- net at R29.1, R30.1, R34.2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: now also C24.1
- net ADC_1 renamed A1
- net A1: now also C21.2
- net ADC_2 renamed A2
- net A2: now also C22.2
- net ADC_3 renamed A3
- net A3: now also C23.2
- net ADC_4 renamed A4
- net A4: now also C24.2
- net ANALOG_IN_1 renamed A1-PRE
- net ANALOG_IN_2 renamed A2-PRE
- net ANALOG_IN_3 renamed A3-PRE
- net ANALOG_IN_4 renamed A4-PRE
- new net: C28.1, R41.1, R42.1, R46.2, U12.13 (-)
- new net: C27.1, R39.1, R40.1, R45.2, U12.9 (-)
- new net: C26.1, R37.1, R38.1, R44.2, U12.6 (-)
- new net: C25.1, R35.1, R36.1, R43.2, U12.2 (-)
- new net: C29.1, R47.1, R48.1, R55.2, U13.2 (-)
- new net: C30.1, R49.1, R50.1, R56.2, U13.6 (-)
- new net: C31.1, R51.1, R52.1, R57.2, U13.9 (-)
- new net: C32.1, R53.1, R54.1, R58.2, U13.13 (-)
- new net +3V3: C18.1, C19.1, C20.1, U11.4 (V+), U12.4 (V+), U13.4 (V+)
- new net A10: C30.2, R56.1, U13.7
- new net A10-PRE: R49.2
- new net A11: C31.2, R57.1, U13.8
- new net A11-PRE: R51.2
- new net A12: C32.2, R58.1, U13.14
- new net A12-PRE: R53.2
- new net A5: C25.2, R43.1, U12.1
- new net A5-PRE: R35.2
- new net A6: C26.2, R44.1, U12.7
- new net A6-PRE: R37.2
- new net A7: C27.2, R45.1, U12.8
- new net A7-PRE: R39.2
- new net A8: C28.2, R46.1, U12.14
- new net A8-PRE: R41.2
- new net A9: C29.2, R55.1, U13.1
- new net A9-PRE: R47.2
Other:
- moved on the sheet: R23, R24, R25, R26, R27, R28, R29, R30, R31, R32, R33, R34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
