File: hardware/AnalogOutBuffers.sch (KiCad schematic (older format))
At the start: 17 parts, among them U10 OPA4197

Commit message: Finish up first plausible version
Parts:
- added C33, C34: 0.1uF, Capacitor_SMD:C_0603_1608Metric_Pad1.08x0.95mm_HandSolder, symbol Device:C_Small
- added unit 5 of U10
- R10, R11, R12, R13, R14, R15, R16, R17, R18, R19, R20, R21, R22, R7, R8, R9: footprint Resistor_SMD:R_0603_1608Metric_Pad1.05x0.95mm_HandSolder -> Resistor_SMD:R_0603_1608Metric_Pad0.98x0.95mm_HandSolder
Connections:
- net DAC_OUT_1: now also R17.1, R21.1; no longer R15.1, R19.1
- net DAC_OUT_2: now also R18.1, R22.1; no longer R16.1, R20.1
- net DAC_OUT_3: now also R15.1, R19.1; no longer R17.1, R21.1
- net DAC_OUT_4: now also R16.1, R20.1; no longer R18.1, R22.1
- net GND: now also C33.1, C34.2
- new net +12V: C34.1, U10.4 (V+)
- new net -12V: C33.2, U10.11 (V-)
Changed lines of the file:
@@
 F 0 "R15" V 1795 1950 50  0000 C CNN
 F 1 "10k" V 1886 1950 50  0000 C CNN
-F 2 "Resistor_SMD:R_0603_1608Metric_Pad1.05x0.95mm_HandSolder" V 2040 1940 50  0001 C CNN
+F 2 "Resistor_SMD:R_0603_1608Metric_Pad0.98x0.95mm_HandSolder" V 2040 1940 50  0001 C CNN
 F 3 "~" H 2000 1950 50  0001 C CNN
 	1    2000 1950
@@
 F 0 "R7" V 1095 1600 50  0000 C CNN
 F 1 "1.54k" V 1186 1600 50  0000 C CNN
-F 2 "Resistor_SMD:R_0603_1608Metric_Pad1.05x0.95mm_HandSolder" V 1340 1590 50  0001 C CNN
+F 2 "Resistor_SMD:R_0603_1608Metric_Pad0.98x0.95mm_HandSolder" V 1340 1590 50  0001 C CNN
 F 3 "~" H 1300 1600 50  0001 C CNN
 	1    1300 1600
@@
 F 0 "R19" V 2220 1500 50  0000 C CNN
 F 1 "1k" V 2311 1500 50  0000 C CNN
-F 2 "Resistor_SMD:R_0603_1608Metric_Pad1.05x0.95mm_HandSolder" V 2465 1490 50  0001 C CNN
+F 2 "Resistor_SMD:R_0603_1608Metric_Pad0.98x0.95mm_HandSolder" V 2465 1490 50  0001 C CNN
 F 3 "~" H 2425 1500 50  0001 C CNN
 	1    2425 1500
@@
 F 0 "R8" V 1095 1950 50  0000 C CNN
 F 1 "12.4k" V 1186 1950 50  0000 C CNN
-F 2 "Resistor_SMD:R_0603_1608Metric_Pad1.05x0.95mm_HandSolder" V 1340 1940 50  0001 C CNN
+F 2 "Resistor_SMD:R_0603_1608Metric_Pad0.98x0.95mm_HandSolder" V 1340 1940 50  0001 C CNN
 F 3 "~" H 1300 1950 50  0001 C CNN
 	1    1300 1950
@@
 F 0 "R16" V 1820 2950 50  0000 C CNN
 F 1 "10k" V 1911 2950 50  0000 C CNN
-F 2 "Resistor_SMD:R_0603_1608Metric_Pad1.05x0.95mm_HandSolder" V 2065 2940 50  0001 C CNN
+F 2 "Resistor_SMD:R_0603_1608Metric_Pad0.98x0.95mm_HandSolder" V 2065 2940 50  0001 C CNN
 F 3 "~" H 2025 2950 50  0001 C CNN
 	1    2025 2950
@@
 F 0 "R9" V 1120 2600 50  0000 C CNN
 F 1 "1.54k" V 1211 2600 50  0000 C CNN
-F 2 "Resistor_SMD:R_0603_1608Metric_Pad1.05x0.95mm_HandSolder" V 1365 2590 50  0001 C CNN
+F 2 "Resistor_SMD:R_0603_1608Metric_Pad0.98x0.95mm_HandSolder" V 1365 2590 50  0001 C CNN
 F 3 "~" H 1325 2600 50  0001 C CNN
 	1    1325 2600
@@
 F 0 "R20" V 2245 2500 50  0000 C CNN
 F 1 "1k" V 2336 2500 50  0000 C CNN
-F 2 "Resistor_SMD:R_0603_1608Metric_Pad1.05x0.95mm_HandSolder" V 2490 2490 50  0001 C CNN
+F 2 "Resistor_SMD:R_0603_1608Metric_Pad0.98x0.95mm_HandSolder" V 2490 2490 50  0001 C CNN
 F 3 "~" H 2450 2500 50  0001 C CNN
 	1    2450 2500
@@
 F 0 "R10" V 1120 2950 50  0000 C CNN
 F 1 "12.4k" V 1211 2950 50  0000 C CNN
-F 2 "Resistor_SMD:R_0603_1608Metric_Pad1.05x0.95mm_HandSolder" V 1365 2940 50  0001 C CNN
+F 2 "Resistor_SMD:R_0603_1608Metric_Pad0.98x0.95mm_HandSolder" V 1365 2940 50  0001 C CNN
 F 3 "~" H 1325 2950 50  0001 C CNN
 	1    1325 2950
@@
 F 0 "R17" V 1820 3925 50  0000 C CNN
 F 1 "10k" V 1911 3925 50  0000 C CNN
-F 2 "Resistor_SMD:R_0603_1608Metric_Pad1.05x0.95mm_HandSolder" V 2065 3915 50  0001 C CNN
+F 2 "Resistor_SMD:R_0603_1608Metric_Pad0.98x0.95mm_HandSolder" V 2065 3915 50  0001 C CNN
 F 3 "~" H 2025 3925 50  0001 C CNN
 	1    2025 3925
@@
 F 0 "R11" V 1120 3575 50  0000 C CNN
 F 1 "1.54k" V 1211 3575 50  0000 C CNN
-F 2 "Resistor_SMD:R_0603_1608Metric_Pad1.05x0.95mm_HandSolder" V 1365 3565 50  0001 C CNN
+F 2 "Resistor_SMD:R_0603_1608Metric_Pad0.98x0.95mm_HandSolder" V 1365 3565 50  0001 C CNN
 F 3 "~" H 1325 3575 50  0001 C CNN
 	1    1325 3575
@@
 F 0 "R21" V 2245 3475 50  0000 C CNN
 F 1 "1k" V 2336 3475 50  0000 C CNN
-F 2 "Resistor_SMD:R_0603_1608Metric_Pad1.05x0.95mm_HandSolder" V 2490 3465 50  0001 C CNN
+F 2 "Resistor_SMD:R_0603_1608Metric_Pad0.98x0.95mm_HandSolder" V 2490 3465 50  0001 C CNN
 F 3 "~" H 2450 3475 50  0001 C CNN
 	1    2450 3475
@@
 F 0 "R12" V 1120 3925 50  0000 C CNN
 F 1 "12.4k" V 1211 3925 50  0000 C CNN
-F 2 "Resistor_SMD:R_0603_1608Metric_Pad1.05x0.95mm_HandSolder" V 1365 3915 50  0001 C CNN
+F 2 "Resistor_SMD:R_0603_1608Metric_Pad0.98x0.95mm_HandSolder" V 1365 3915 50  0001 C CNN
 F 3 "~" H 1325 3925 50  0001 C CNN
 	1    1325 3925
@@
 F 0 "R18" V 1820 4900 50  0000 C CNN
 F 1 "10k" V 1911 4900 50  0000 C CNN
-F 2 "Resistor_SMD:R_0603_1608Metric_Pad1.05x0.95mm_HandSolder" V 2065 4890 50  0001 C CNN
+F 2 "Resistor_SMD:R_0603_1608Metric_Pad0.98x0.95mm_HandSolder" V 2065 4890 50  0001 C CNN
 F 3 "~" H 2025 4900 50  0001 C CNN
 	1    2025 4900
@@
 F 0 "R13" V 1120 4550 50  0000 C CNN
 F 1 "1.54k" V 1211 4550 50  0000 C CNN
-F 2 "Resistor_SMD:R_0603_1608Metric_Pad1.05x0.95mm_HandSolder" V 1365 4540 50  0001 C CNN
+F 2 "Resistor_SMD:R_0603_1608Metric_Pad0.98x0.95mm_HandSolder" V 1365 4540 50  0001 C CNN
 F 3 "~" H 1325 4550 50  0001 C CNN
 	1    1325 4550
@@
 F 0 "R22" V 2245 4450 50  0000 C CNN
 F 1 "1k" V 2336 4450 50  0000 C CNN
-F 2 "Resistor_SMD:R_0603_1608Metric_Pad1.05x0.95mm_HandSolder" V 2490 4440 50  0001 C CNN
+F 2 "Resistor_SMD:R_0603_1608Metric_Pad0.98x0.95mm_HandSolder" V 2490 4440 50  0001 C CNN
 F 3 "~" H 2450 4450 50  0001 C CNN
 	1    2450 4450
@@
 F 0 "R14" V 1120 4900 50  0000 C CNN
 F 1 "12.4k" V 1211 4900 50  0000 C CNN
-F 2 "Resistor_SMD:R_0603_1608Metric_Pad1.05x0.95mm_HandSolder" V 1365 4890 50  0001 C CNN
+F 2 "Resistor_SMD:R_0603_1608Metric_Pad0.98x0.95mm_HandSolder" V 1365 4890 50  0001 C CNN
 F 3 "~" H 1325 4900 50  0001 C CNN
 	1    1325 4900
@@
 Text Notes 825  4475 0    50   ~ 0
 0 - 2.5v
-Text HLabel 1150 1600 0    50   Input ~ 0
-DAC_IN_1
 Text HLabel 1175 2600 0    50   Input ~ 0
 DAC_IN_2
 Text HLabel 1175 3575 0    50   Input ~ 0
 DAC_IN_3
+Text HLabel 2600 3475 2    50   Input ~ 0
+DAC_OUT_1
+Text HLabel 2600 4450 2    50   Input ~ 0
+DAC_OUT_2
+Text HLabel 2575 1500 2    50   Input ~ 0
+DAC_OUT_3
+Text HLabel 2600 2500 2    50   Input ~ 0
+DAC_OUT_4
+$Comp
+L winterbloom:OPA4197 U10
+U 5 1 61594009
+P 4625 2050
+F 0 "U10" H 4650 2225 50  0000 C CNN
+F 1 "OPA4197" H 4750 1875 50  0000 C CNN
+F 2 "Package_SO:TSSOP-14_4.4x5mm_P0.65mm" H 4625 1700 50  0001 C CNN
+F 3 "https://www.ti.com/lit/ds/symlink/opa4197.pdf" H 4675 2250 50  0001 C CNN
+F 4 "OPA4197IPW" H 4625 1600 39  0001 C CNN "mpn"
+	5    4625 2050
+	1    0    0    -1
+$EndComp
+$Comp
+L power:-12V #PWR0161
+U 1 1 61595B3A
+P 4525 2350
+F 0 "#PWR0161" H 4525 2450 50  0001 C CNN
+F 1 "-12V" H 4540 2523 50  0000 C CNN
+F 2 "" H 4525 2350 50  0001 C CNN
+F 3 "" H 4525 2350 50  0001 C CNN
+	1    4525 2350
+	-1   0    0    1
+$EndComp
+$Comp
+L power:+12V #PWR0162
+U 1 1 61596478
+P 4525 1750
+F 0 "#PWR0162" H 4525 1600 50  0001 C CNN
+F 1 "+12V" H 4540 1923 50  0000 C CNN
+F 2 "" H 4525 1750 50  0001 C CNN
+F 3 "" H 4525 1750 50  0001 C CNN
+	1    4525 1750
+	1    0    0    -1
+$EndComp
+$Comp
+L power:+12V #PWR0163
+U 1 1 615968CE
+P 5875 2075
+F 0 "#PWR0163" H 5875 1925 50  0001 C CNN
+F 1 "+12V" H 5890 2248 50  0000 C CNN
+F 2 "" H 5875 2075 50  0001 C CNN
+F 3 "" H 5875 2075 50  0001 C CNN
+	1    5875 2075
+	1    0    0    -1
+$EndComp
+$Comp
+L power:-12V #PWR0164
+U 1 1 61596B9E
+P 5450 2175
+F 0 "#PWR0164" H 5450 2275 50  0001 C CNN
+F 1 "-12V" H 5465 2348 50  0000 C CNN
+F 2 "" H 5450 2175 50  0001 C CNN
+F 3 "" H 5450 2175 50  0001 C CNN
+	1    5450 2175
+	-1   0    0    1
+$EndComp
+$Comp
+L Device:C_Small C33
+U 1 1 615973E7
+P 5450 2075
+F 0 "C33" H 5542 2121 50  0000 L CNN
+F 1 "0.1uF" H 5542 2030 50  0000 L CNN
+F 2 "Capacitor_SMD:C_0603_1608Metric_Pad1.08x0.95mm_HandSolder" H 5450 2075 50  0001 C CNN
+F 3 "~" H 5450 2075 50  0001 C CNN
+	1    5450 2075
+	1    0    0    -1
+$EndComp
+$Comp
+L Device:C_Small C34
+U 1 1 61597F9E
+P 5875 2175
+F 0 "C34" H 5967 2221 50  0000 L CNN
+F 1 "0.1uF" H 5967 2130 50  0000 L CNN
+F 2 "Capacitor_SMD:C_0603_1608Metric_Pad1.08x0.95mm_HandSolder" H 5875 2175 50  0001 C CNN
+F 3 "~" H 5875 2175 50  0001 C CNN
+	1    5875 2175
+	1    0    0    -1
+$EndComp
+$Comp
+L power:GND #PWR0165
+U 1 1 61598D1B
+P 5450 1975
+F 0 "#PWR0165" H 5450 1725 50  0001 C CNN
+F 1 "GND" H 5455 1802 50  0001 C CNN
+F 2 "" H 5450 1975 50  0001 C CNN
+F 3 "" H 5450 1975 50  0001 C CNN
+	1    5450 1975
+	-1   0    0    1
+$EndComp
+$Comp
+L power:GND #PWR0166
+U 1 1 61599110
+P 5875 2275
+F 0 "#PWR0166" H 5875 2025 50  0001 C CNN
+F 1 "GND" H 5880 2102 50  0001 C CNN
+F 2 "" H 5875 2275 50  0001 C CNN
+F 3 "" H 5875 2275 50  0001 C CNN
+	1    5875 2275
+	1    0    0    -1
+$EndComp
 Text HLabel 1175 4550 0    50   Input ~ 0
 DAC_IN_4
-Text HLabel 2575 1500 2    50   Input ~ 0
-DAC_OUT_1
-Text HLabel 2600 2500 2    50   Input ~ 0
-DAC_OUT_2
-Text HLabel 2600 3475 2    50   Input ~ 0
-DAC_OUT_3
-Text HLabel 2600 4450 2    50   Input ~ 0
-DAC_OUT_4
+Text HLabel 1150 1600 0    50   Input ~ 0
+DAC_IN_1
 $EndSCHEMATC
