File: hardware/mcu.sch (KiCad schematic (older format))
At the start: 21 parts, among them J3 USB_B, J4 Tag-Connect_SWD_TC2030, SW2 Reset, U5 ATSAMD51J20A-M, U6 AD5685R?RUZ, Y1 32.768 kHz

Commit message: Finish up first plausible version
Parts:
- removed JP1: FS0, Jumper:SolderJumper-2_P1.3mm_Bridged_RoundedPad1.0x1.5mm, symbol Jumper:SolderJumper_2_Bridged
- removed JP2: FS1, Jumper:SolderJumper-2_P1.3mm_Open_RoundedPad1.0x1.5mm, symbol Jumper:SolderJumper_2_Open
- added C15, C16: 0.1uF, Capacitor_SMD:C_0603_1608Metric_Pad1.08x0.95mm_HandSolder, symbol Device:C_Small
- added C17: 1uF, Capacitor_SMD:C_0603_1608Metric_Pad1.08x0.95mm_HandSolder, symbol Device:C_Small
- added R59, R60: 1k, Resistor_SMD:R_0603_1608Metric_Pad0.98x0.95mm_HandSolder, symbol Device:R_US
- C10, C11, C12, C13, C14, C6, C7, C8, C9: footprint Capacitor_SMD:C_0603_1608Metric_Pad1.05x0.95mm_HandSolder -> Capacitor_SMD:C_0603_1608Metric_Pad1.08x0.95mm_HandSolder
- J3: symbol Connector:USB_B -> testkit-rescue:USB_B-Connector
- R4: footprint Resistor_SMD:R_0603_1608Metric_Pad1.05x0.95mm_HandSolder -> Resistor_SMD:R_0603_1608Metric_Pad0.98x0.95mm_HandSolder
- Y1: footprint Crystal:Crystal_SMD_Abracon_ABM3-2Pin_5.0x3.2mm_HandSoldering -> Crystal:Crystal_SMD_2012-2Pin_2.0x1.2mm_HandSoldering
Connections:
- net DAC_SCLK is gone; now on net SPI_SCLK: U6.12 (SCLK)
- net DAC_SDIN is gone; now on net SPI_COPI: U6.14 (SDIN)
- net +3V3: now also FB4.2, C15.1, R59.1, R60.1; no longer FB4.1
- net DAC_CS: now also U5.31 (PA14)
- net DOTSTAR_CI: now also U5.44 (PA23)
- net DOTSTAR_DI: now also U5.43 (PA22)
- net GND: now also C15.2, C16.2, C17.2
- net RESET: now also U5.52 (~RESET)
- net A10: now reaches U5.10 (PB07)
- net A11: now reaches U5.11 (PB08)
- net A12: now reaches U5.12 (PB09)
- net A13: now reaches U5.13 (PA04)
- net A14: now reaches U5.14 (PA05)
- net A15: now reaches U5.15 (PA06)
- net A16: now reaches U5.16 (PA07)
- net SERIAL4.2: now reaches U5.27 (PB14)
- net SERIAL4.3: now reaches U5.28 (PB15)
- net DB0: now reaches U5.29 (PA12)
- net A5: now reaches U5.3 (PA02)
- net SPI_SCLK: now reaches U5.30 (PA13)
- net SPI_COPI: now reaches U5.32 (PA15)
- net SERIAL1.0: now reaches U5.35 (PA16)
- net SERIAL1.1: now reaches U5.36 (PA17)
- net SERIAL1.2: now reaches U5.37 (PA18)
- net SERIAL1.3: now reaches U5.38 (PA19)
- net DR4: now reaches U5.39 (PB16)
- net A6: now reaches U5.4 (PA03)
- net DR3: now reaches U5.40 (PB17)
- net DR2: now reaches U5.41 (PA20)
- net DR1: now reaches U5.42 (PA21)
- net PB22: now reaches U5.49 (PB22)
- net A7: now reaches U5.5 (PB04)
- net PB23: now reaches U5.50 (PB23)
- net PA27: now reaches U5.51 (PA27)
- net I2C_SDA: now reaches U5.59 (PB30)
- net I2C_SDA: now also R59.2
- net A8: now reaches U5.6 (PB05)
- net I2C_SCL: now reaches U5.60 (PB31)
- net I2C_SCL: now also R60.2
- net A1: now reaches U5.61 (PB00)
- net A2: now reaches U5.62 (PB01)
- net A3: now reaches U5.63 (PB02)
- net A4: now reaches U5.64 (PB03)
- net A9: now reaches U5.9 (PB06)
- net at U6.5 (VDD): now also FB4.1, C16.1, C17.1; no longer FB4.2
- net I2S_FS1 renamed DB2
- net I2S_IN_SD renamed DB1
- net I2S_MCK1 renamed SERIAL4.1
- net I2S_MCLK renamed A18
- net I2S_OUT_SD renamed A19
- net I2S_OUT_WS renamed A17
- net I2S_SCK renamed A20
- net I2S_SCK1 renamed SERIAL4.0
Other:
- note added: "2.1, 2.2, 2.3 used by DAC"
- note added: "3.0, 3.1 used by dotstar"
- note added: "5.0, 5.1 used by I2C"
- note removed: "Needs bypass caps"
- note removed: "TODO"
- moved on the sheet: D3, FB4, U6
