File: hardware/switching.sch (KiCad schematic (older format))
At the start: 5 parts, among them U7 ADG1414BRU, U8 ADG1414BRU, U9 ADG1414BRU

Commit message: Finish up first plausible version
Parts:
- R5, R6: footprint Resistor_SMD:R_0603_1608Metric_Pad1.05x0.95mm_HandSolder -> Resistor_SMD:R_0603_1608Metric_Pad0.98x0.95mm_HandSolder
Connections:
- net ADC_1 is gone; now on net DAC_3: U9.11 (S4), U9.5 (S1), U9.7 (S2), U9.9 (S3)
- net ADC_1A is gone; now on net DAC_3A: U9.6 (D1)
- net ADC_1B is gone; now on net DAC_3B: U9.8 (D2)
- net ADC_2 is gone; now on net DAC_4: U9.14 (S5), U9.16 (S6), U9.18 (S7), U9.20 (S8)
- net ADC_2A is gone; now on net DAC_4A: U9.13 (D5)
- net ADC_2B is gone; now on net DAC_4B: U9.15 (D6)
- net DAC_1: now also U8.11 (S4), U8.9 (S3)
- net DAC_2: now also U8.14 (S5), U8.16 (S6), U8.18 (S7), U8.20 (S8); no longer U8.11 (S4), U8.9 (S3)
- net DAC_2A: now also U8.13 (D5); no longer U8.10 (D3)
- net DAC_2B: now also U8.15 (D6); no longer U8.12 (D4)
- net DAC_3: no longer U8.14 (S5), U8.16 (S6)
- net DAC_3A: no longer U8.13 (D5)
- net DAC_3B: no longer U8.15 (D6)
- net DAC_4: no longer U8.18 (S7), U8.20 (S8)
- net DAC_4A: no longer U8.17 (D7)
- net DAC_4B: no longer U8.19 (D8)
- net ADC_1C renamed DAC_3C
- net ADC_1D renamed DAC_3D
- net ADC_2C renamed DAC_4C
- net ADC_2D renamed DAC_4D
- new net DAC_1C: U8.10 (D3)
- new net DAC_1D: U8.12 (D4)
- new net DAC_2C: U8.17 (D7)
- new net DAC_2D: U8.19 (D8)
- no-connect marks 0 -> 1
Other:
- note added: "Analog out 2:8 multiplexer"
- note added: "bypass caps?"
- note removed: "Analog out 4:8 multiplexer"
Changed lines of the file:
@@
 	1    0    0    -1
 $EndComp
-Text HLabel 8750 2150 2    50   Input ~ 0
-ADC_2D
-Text HLabel 8750 2050 2    50   Input ~ 0
-ADC_2C
-Text HLabel 8750 1950 2    50   Input ~ 0
-ADC_2B
-Text HLabel 8750 1850 2    50   Input ~ 0
-ADC_2A
-Text HLabel 8750 1750 2    50   Input ~ 0
-ADC_1D
-Text HLabel 8750 1650 2    50   Input ~ 0
-ADC_1C
-Text HLabel 8750 1550 2    50   Input ~ 0
-ADC_1B
-Text HLabel 8750 1450 2    50   Input ~ 0
-ADC_1A
-Connection ~ 7150 2050
-Wire Wire Line
-	7150 2050 7150 2150
-Connection ~ 7150 1950
-Wire Wire Line
-	7150 1950 7150 2050
-Wire Wire Line
-	7150 1850 7150 1950
-Text HLabel 7150 1850 0    50   Input ~ 0
-ADC_2
-Connection ~ 7150 1650
-Wire Wire Line
-	7150 1650 7150 1750
-Connection ~ 7150 1550
-Wire Wire Line
-	7150 1550 7150 1650
-Wire Wire Line
-	7150 1450 7150 1550
-Text HLabel 7150 1450 0    50   Input ~ 0
-ADC_1
 Text Notes 7400 850  0    50   ~ 0
 Analog in 2:8 multiplexer
@@
 $EndComp
 Text HLabel 5775 2175 2    50   Input ~ 0
-DAC_4B
+DAC_2D
 Text HLabel 5775 2075 2    50   Input ~ 0
-DAC_4A
+DAC_2C
 Text HLabel 5775 1975 2    50   Input ~ 0
-DAC_3B
+DAC_2B
 Text HLabel 5775 1875 2    50   Input ~ 0
-DAC_3A
+DAC_2A
 Text HLabel 5775 1775 2    50   Input ~ 0
-DAC_2B
+DAC_1D
 Text HLabel 5775 1675 2    50   Input ~ 0
-DAC_2A
+DAC_1C
 Text HLabel 5775 1575 2    50   Input ~ 0
 DAC_1B
 Text HLabel 5775 1475 2    50   Input ~ 0
 DAC_1A
-Wire Wire Line
-	4175 2075 4175 2175
-Wire Wire Line
-	4175 1875 4175 1975
-Wire Wire Line
-	4175 1675 4175 1775
-Text HLabel 4175 2075 0    50   Input ~ 0
-DAC_4
 Text HLabel 4175 1875 0    50   Input ~ 0
-DAC_3
-Text HLabel 4175 1675 0    50   Input ~ 0
 DAC_2
 Wire Wire Line
@@
 DAC_1
 Text Notes 4425 850  0    50   ~ 0
-Analog out 4:8 multiplexer
+Analog out 2:8 multiplexer
 $Comp
 L Analog_Switch:ADG1414BRU U?
@@
 F 0 "R5" H 3693 2371 50  0000 L CNN
 F 1 "1k" H 3693 2280 50  0000 L CNN
-F 2 "Resistor_SMD:R_0603_1608Metric_Pad1.05x0.95mm_HandSolder" V 3665 2315 50  0001 C CNN
+F 2 "Resistor_SMD:R_0603_1608Metric_Pad0.98x0.95mm_HandSolder" V 3665 2315 50  0001 C CNN
 F 3 "~" H 3625 2325 50  0001 C CNN
 	1    3625 2325
@@
 F 0 "R6" H 6668 2346 50  0000 L CNN
 F 1 "1k" H 6668 2255 50  0000 L CNN
-F 2 "Resistor_SMD:R_0603_1608Metric_Pad1.05x0.95mm_HandSolder" V 6640 2290 50  0001 C CNN
+F 2 "Resistor_SMD:R_0603_1608Metric_Pad0.98x0.95mm_HandSolder" V 6640 2290 50  0001 C CNN
 F 3 "~" H 6600 2300 50  0001 C CNN
 	1    6600 2300
@@
 Wire Wire Line
 	4175 3350 4175 2775
+Wire Wire Line
+	4175 1575 4175 1675
+Connection ~ 4175 1575
+Wire Wire Line
+	4175 1675 4175 1775
+Connection ~ 4175 1675
+Wire Wire Line
+	4175 1875 4175 1975
+Wire Wire Line
+	4175 1975 4175 2075
+Connection ~ 4175 1975
+Wire Wire Line
+	4175 2075 4175 2175
+Connection ~ 4175 2075
+Text HLabel 7150 1450 0    50   Input ~ 0
+DAC_3
+Text HLabel 7150 1850 0    50   Input ~ 0
+DAC_4
+Wire Wire Line
+	7150 1450 7150 1550
+Wire Wire Line
+	7150 1550 7150 1650
+Connection ~ 7150 1550
+Wire Wire Line
+	7150 1650 7150 1750
+Connection ~ 7150 1650
+Wire Wire Line
+	7150 1850 7150 1950
+Wire Wire Line
+	7150 1950 7150 2050
+Connection ~ 7150 1950
+Wire Wire Line
+	7150 2050 7150 2150
+Connection ~ 7150 2050
+Text HLabel 8750 2150 2    50   Input ~ 0
+DAC_4D
+Text HLabel 8750 2050 2    50   Input ~ 0
+DAC_4C
+Text HLabel 8750 1950 2    50   Input ~ 0
+DAC_4B
+Text HLabel 8750 1850 2    50   Input ~ 0
+DAC_4A
+Text HLabel 8750 1750 2    50   Input ~ 0
+DAC_3D
+Text HLabel 8750 1650 2    50   Input ~ 0
+DAC_3C
+Text HLabel 8750 1550 2    50   Input ~ 0
+DAC_3B
+Text HLabel 8750 1450 2    50   Input ~ 0
+DAC_3A
+Text Notes 6050 950  0    50   ~ 0
+bypass caps?
+NoConn ~ 7150 2750
 $EndSCHEMATC
