File: hardware/testkit.kicad_pcb (KiCad board)
At the start: 2 copper layers, 100 x 100 mm, 97 parts, among them J1 Eurorack_Power, J3 USB_B, J4 Tag-Connect_SWD_TC2030, J5 Left, J6 Right, J7 Top, SW2 Reset, U1 INA219BxDCN, U10 OPA4197, U11 MCP6004, U12 SSM2604, U2 INA219BxDCN, U3 TLV76733, U4 LM4040-10, U5 ATSAMD51J20A-M, U6 AD5685R?RUZ, U7 ADG1414BRU, U8 ADG1414BRU, U9 ADG1414BRU, Y1 32.768 kHz, Y2 12.228 MHz

Commit message: Finish up first plausible version
Parts:
- removed FB5, FB6: 300mA, Inductor_SMD:L_0603_1608Metric_Pad1.05x0.95mm_HandSolder
- removed JP1: FS0, Jumper:SolderJumper-2_P1.3mm_Bridged_RoundedPad1.0x1.5mm
- removed JP2: FS1, Jumper:SolderJumper-2_P1.3mm_Open_RoundedPad1.0x1.5mm
- removed JP3: MCLKSEL, Jumper:SolderJumper-3_P1.3mm_Bridged12_RoundedPad1.0x1.5mm
- removed Y2: 12.228 MHz, Crystal:Crystal_SMD_Abracon_ABM3-2Pin_5.0x3.2mm_HandSoldering
- added C25: 22pF, Capacitor_SMD:C_0603_1608Metric_Pad1.08x0.95mm_HandSolder, F.Cu at (93.0, 101.9)
- added C26: 22pF, Capacitor_SMD:C_0603_1608Metric_Pad1.08x0.95mm_HandSolder, F.Cu at (93.0, 107.9)
- added C27: 22pF, Capacitor_SMD:C_0603_1608Metric_Pad1.08x0.95mm_HandSolder, F.Cu at (108.1, 107.0)
- added C28: 22pF, Capacitor_SMD:C_0603_1608Metric_Pad1.08x0.95mm_HandSolder, F.Cu at (108.1, 103.0)
- added C29: 22pF, Capacitor_SMD:C_0603_1608Metric_Pad1.08x0.95mm_HandSolder, F.Cu at (92.8, 113.0)
- added C30: 22pF, Capacitor_SMD:C_0603_1608Metric_Pad1.08x0.95mm_HandSolder, F.Cu at (93.0, 119.0)
- added C31: 22pF, Capacitor_SMD:C_0603_1608Metric_Pad1.08x0.95mm_HandSolder, F.Cu at (108.1, 117.9)
- added C32: 22pF, Capacitor_SMD:C_0603_1608Metric_Pad1.08x0.95mm_HandSolder, F.Cu at (108.1, 114.0)
- added C33: 0.1uF, Capacitor_SMD:C_0603_1608Metric_Pad1.08x0.95mm_HandSolder, F.Cu at (148.4, 110.7)
- added C34: 0.1uF, Capacitor_SMD:C_0603_1608Metric_Pad1.08x0.95mm_HandSolder, F.Cu at (148.4, 124.0)
- added J12: OSC A, Connector_Audio:Jack_3.5mm_CUI_SJ1-3533NG_Horizontal, F.Cu at (114.0, 51.4)
- added J13: OSC B, Connector_Audio:Jack_3.5mm_CUI_SJ1-3533NG_Horizontal, F.Cu at (123.6, 51.5)
- added J14: OSC C, Connector_Audio:Jack_3.5mm_CUI_SJ1-3533NG_Horizontal, F.Cu at (133.3, 51.5)
- added J15: OSC D, Connector_Audio:Jack_3.5mm_CUI_SJ1-3533NG_Horizontal, F.Cu at (143.0, 51.5)
- added J8: AUDIO IN, Connector_Audio:Jack_3.5mm_CUI_SJ1-3533NG_Horizontal, F.Cu at (152.6, 51.5)
- added J9: AUDIO OUT, Connector_Audio:Jack_3.5mm_CUI_SJ1-3533NG_Horizontal, F.Cu at (162.3, 51.5)
- added R41: 100k, Resistor_SMD:R_0603_1608Metric_Pad0.98x0.95mm_HandSolder, F.Cu at (110.2, 103.0)
- added R42: 121k, Resistor_SMD:R_0603_1608Metric_Pad0.98x0.95mm_HandSolder, F.Cu at (112.3, 103.0)
- added R43: 18.7k, Resistor_SMD:R_0603_1608Metric_Pad0.98x0.95mm_HandSolder, F.Cu at (95.0, 101.9)
- added R44: 18.7k, Resistor_SMD:R_0603_1608Metric_Pad0.98x0.95mm_HandSolder, F.Cu at (95.0, 107.9)
- added R45: 18.7k, Resistor_SMD:R_0603_1608Metric_Pad0.98x0.95mm_HandSolder, F.Cu at (106.0, 107.0)
- added R46: 18.7k, Resistor_SMD:R_0603_1608Metric_Pad0.98x0.95mm_HandSolder, F.Cu at (106.0, 103.0)
- added R47: 100k, Resistor_SMD:R_0603_1608Metric_Pad0.98x0.95mm_HandSolder, F.Cu at (90.8, 113.0)
- added R48: 121k, Resistor_SMD:R_0603_1608Metric_Pad0.98x0.95mm_HandSolder, F.Cu at (88.7, 113.0)
- added R49: 100k, Resistor_SMD:R_0603_1608Metric_Pad0.98x0.95mm_HandSolder, F.Cu at (90.8, 119.0)
- added R50: 121k, Resistor_SMD:R_0603_1608Metric_Pad0.98x0.95mm_HandSolder, F.Cu at (88.7, 119.0)
- added R51: 100k, Resistor_SMD:R_0603_1608Metric_Pad0.98x0.95mm_HandSolder, F.Cu at (110.2, 117.9)
- added R52: 121k, Resistor_SMD:R_0603_1608Metric_Pad0.98x0.95mm_HandSolder, F.Cu at (112.3, 117.9)
- added R53: 100k, Resistor_SMD:R_0603_1608Metric_Pad0.98x0.95mm_HandSolder, F.Cu at (110.2, 114.0)
- added R54: 121k, Resistor_SMD:R_0603_1608Metric_Pad0.98x0.95mm_HandSolder, F.Cu at (112.3, 114.0)
- added R55: 18.7k, Resistor_SMD:R_0603_1608Metric_Pad0.98x0.95mm_HandSolder, F.Cu at (95.0, 113.0)
- added R56: 18.7k, Resistor_SMD:R_0603_1608Metric_Pad0.98x0.95mm_HandSolder, F.Cu at (95.0, 119.0)
- added R57: 18.7k, Resistor_SMD:R_0603_1608Metric_Pad0.98x0.95mm_HandSolder, F.Cu at (106.0, 117.9)
- added R58: 18.7k, Resistor_SMD:R_0603_1608Metric_Pad0.98x0.95mm_HandSolder, F.Cu at (106.0, 114.0)
- added R59: 1k, Resistor_SMD:R_0603_1608Metric_Pad0.98x0.95mm_HandSolder, F.Cu at (100.6, 72.1)
- added R60: 1k, Resistor_SMD:R_0603_1608Metric_Pad0.98x0.95mm_HandSolder, F.Cu at (102.8, 72.1)
- added REF**: MountingHole_3.2mm_M3, MountingHole:MountingHole_3.2mm_M3, F.Cu at (80.0, 144.0)
- added REF**: MountingHole_3.2mm_M3, MountingHole:MountingHole_3.2mm_M3, F.Cu at (170.0, 144.0)
- added REF**: MountingHole_3.2mm_M3, MountingHole:MountingHole_3.2mm_M3, F.Cu at (80.0, 54.0)
- added REF**: MountingHole_3.2mm_M3, MountingHole:MountingHole_3.2mm_M3, F.Cu at (170.0, 54.0)
- added SW1: POWER, Connector_PinSocket_2.54mm:PinSocket_2x02_P2.54mm_Vertical, F.Cu at (91.0, 80.8)
- added U13: MCP6004, Package_SO:TSSOP-14_4.4x5mm_P0.65mm, F.Cu at (100.6, 116.0)
- C1, C4: footprint Capacitor_SMD:C_0603_1608Metric_Pad1.05x0.95mm_HandSolder -> Capacitor_SMD:C_0805_2012Metric_Pad1.18x1.45mm_HandSolder
- C10, C11, C12, C13, C14, C18, C2, C3, C5, C6, C7, C8, C9: footprint Capacitor_SMD:C_0603_1608Metric_Pad1.05x0.95mm_HandSolder -> Capacitor_SMD:C_0603_1608Metric_Pad1.08x0.95mm_HandSolder
- C15, C16: value 22pF -> 0.1uF; footprint Capacitor_SMD:C_0603_1608Metric_Pad1.05x0.95mm_HandSolder -> Capacitor_SMD:C_0603_1608Metric_Pad1.08x0.95mm_HandSolder
- C17: value 4.7uF -> 1uF; footprint Capacitor_SMD:C_0603_1608Metric_Pad1.05x0.95mm_HandSolder -> Capacitor_SMD:C_0603_1608Metric_Pad1.08x0.95mm_HandSolder
- C19, C20: value 1uF -> 0.1uF; footprint Capacitor_SMD:C_0603_1608Metric_Pad1.05x0.95mm_HandSolder -> Capacitor_SMD:C_0603_1608Metric_Pad1.08x0.95mm_HandSolder
- C21, C22: value 1uF -> 22pF; footprint Capacitor_SMD:C_0603_1608Metric_Pad1.05x0.95mm_HandSolder -> Capacitor_SMD:C_0603_1608Metric_Pad1.08x0.95mm_HandSolder
- C23, C24: value 220pF -> 22pF; footprint Capacitor_SMD:C_0603_1608Metric_Pad1.05x0.95mm_HandSolder -> Capacitor_SMD:C_0603_1608Metric_Pad1.08x0.95mm_HandSolder
- J1: value Eurorack_Power -> Power; footprint winterbloom:Eurorack_Power -> Connector_PinHeader_2.54mm:PinHeader_2x05_P2.54mm_Horizontal
- J7: value Top -> Bottom
- R1, R2: footprint Resistor_SMD:R_0603_1608Metric_Pad1.05x0.95mm_HandSolder -> Resistor_SMD:R_1210_3225Metric_Pad1.30x2.65mm_HandSolder
- R10, R11, R12, R13, R14, R15, R16, R17, R18, R19, R20, R21, R22, R23, R24, R25, R26, R27, R28, R29, R3, R30, R31, R32, R33, R34, R4, R5, R6, R7, R8, R9: footprint Resistor_SMD:R_0603_1608Metric_Pad1.05x0.95mm_HandSolder -> Resistor_SMD:R_0603_1608Metric_Pad0.98x0.95mm_HandSolder
- R35: value 47k -> 100k; footprint Resistor_SMD:R_0603_1608Metric_Pad1.05x0.95mm_HandSolder -> Resistor_SMD:R_0603_1608Metric_Pad0.98x0.95mm_HandSolder
- R36: value 47k -> 121k; footprint Resistor_SMD:R_0603_1608Metric_Pad1.05x0.95mm_HandSolder -> Resistor_SMD:R_0603_1608Metric_Pad0.98x0.95mm_HandSolder
- R37: value 5.6k -> 100k; footprint Resistor_SMD:R_0603_1608Metric_Pad1.05x0.95mm_HandSolder -> Resistor_SMD:R_0603_1608Metric_Pad0.98x0.95mm_HandSolder
- R38: value 5.6k -> 121k; footprint Resistor_SMD:R_0603_1608Metric_Pad1.05x0.95mm_HandSolder -> Resistor_SMD:R_0603_1608Metric_Pad0.98x0.95mm_HandSolder
- R39: value 100 -> 100k; footprint Resistor_SMD:R_0805_2012Metric_Pad1.15x1.40mm_HandSolder -> Resistor_SMD:R_0603_1608Metric_Pad0.98x0.95mm_HandSolder
- R40: value 100 -> 121k; footprint Resistor_SMD:R_0805_2012Metric_Pad1.15x1.40mm_HandSolder -> Resistor_SMD:R_0603_1608Metric_Pad0.98x0.95mm_HandSolder
- U12: value SSM2604 -> MCP6004; footprint Package_CSP:LFCSP-20-1EP_4x4mm_P0.5mm_EP2.6x2.6mm -> Package_SO:TSSOP-14_4.4x5mm_P0.65mm
- U3: footprint Package_SO:VSSOP-8_3.0x3.0mm_P0.65mm -> winterbloom:TI-DGN-HVSSOP-8_3.0x3.0mm_P0.65mm
- Y1: footprint Crystal:Crystal_SMD_Abracon_ABM3-2Pin_5.0x3.2mm_HandSoldering -> Crystal:Crystal_SMD_2012-2Pin_2.0x1.2mm_HandSoldering
- moved SW2 237.9 mm to (131.6, 87.8)
- moved C17 207.8 mm to (138.1, 111.1), turned to 90 degrees
- moved C16 204.3 mm to (140.1, 111.4), turned to 90 degrees
- moved R20 203.4 mm to (151.6, 123.1), turned to 180 degrees
- moved C12 199.2 mm to (137.6, 97.3)
- moved C14 198.6 mm to (137.6, 106.0)
- moved R21 197.2 mm to (151.6, 111.1), turned to 180 degrees
- moved C9 195.5 mm to (133.7, 93.9), turned to 90 degrees
- moved R22 195.2 mm to (145.2, 111.1)
- moved C15 193.3 mm to (137.0, 121.2)
- moved R39 192.8 mm to (110.2, 107.0), turned to 270 degrees
- moved FB4 192.4 mm to (136.1, 111.4), turned to 270 degrees
- moved R40 187.5 mm to (112.3, 107.0), turned to 90 degrees
- moved C13 187.5 mm to (129.7, 93.9), turned to 90 degrees
- moved C23 186.3 mm to (108.1, 96.0), turned to 270 degrees
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Connections:
- net /MCU/DAC_1 renamed DAC_1
- net /MCU/DAC_2 renamed DAC_2
- net /MCU/DAC_3 renamed DAC_3
- net /MCU/DAC_4 renamed DAC_4
- net Net-(U5-Pad49) renamed /MCU/PB22
- net Net-(U5-Pad50) renamed /MCU/PB23
- net Net-(U5-Pad51) renamed /MCU/PA27
- C15 pad 1: /CODEC/XTI -> +3V3
- C16 pad 1: /CODEC/XTO -> Net-(C16-Pad1)
- C17 pad 1: Net-(C17-Pad1) -> Net-(C16-Pad1)
- C18 pad 1: Net-(C17-Pad1) -> +3V3
- C19 pad 1: Net-(C19-Pad1) -> +3V3
- C19 pad 2: Net-(C19-Pad2) -> GND
- C20 pad 1: Net-(C20-Pad1) -> +3V3
- C20 pad 2: Net-(C20-Pad2) -> GND
- C21 pad 2: Net-(C21-Pad2) -> A1
- C22 pad 2: Net-(C22-Pad2) -> A2
- C23 pad 1: GND -> Net-(C23-Pad1)
- C23 pad 2: Net-(C21-Pad1) -> A3
- C24 pad 1: GND -> Net-(C24-Pad1)
- C24 pad 2: Net-(C22-Pad1) -> A4
- C5 pad 2: Net-(C5-Pad2) -> -10V
- D1 pad 2: +12V -> -12V
- D2 pad 1: -12V -> +12V
- FB4 pad 1: +3V3 -> Net-(C16-Pad1)
- FB4 pad 2: Net-(FB4-Pad2) -> +3V3
- J5 pad 1: Net-(J5-Pad1) -> GND
- J5 pad 10: Net-(J5-Pad10) -> GND
- J5 pad 11: Net-(J5-Pad11) -> +3V3
- J5 pad 12: Net-(J5-Pad12) -> +3V3
- J5 pad 13: Net-(J5-Pad13) -> GND
- J5 pad 14: Net-(J5-Pad14) -> GND
- J5 pad 15: Net-(J5-Pad15) -> A1-PRE
- J5 pad 16: Net-(J5-Pad16) -> A2-PRE
- J5 pad 17: Net-(J5-Pad17) -> A3-PRE
- J5 pad 18: Net-(J5-Pad18) -> A4-PRE
- J5 pad 19: Net-(J5-Pad19) -> A5-PRE
- J5 pad 2: Net-(J5-Pad2) -> GND
- J5 pad 20: Net-(J5-Pad20) -> A6-PRE
- J5 pad 21: Net-(J5-Pad21) -> A7-PRE
- J5 pad 22: Net-(J5-Pad22) -> A8-PRE
- J5 pad 23: Net-(J5-Pad23) -> A9-PRE
- J5 pad 24: Net-(J5-Pad24) -> A10-PRE
- J5 pad 25: Net-(J5-Pad25) -> A11-PRE
- J5 pad 26: Net-(J5-Pad26) -> A12-PRE
- J5 pad 27: Net-(J5-Pad27) -> GND
- J5 pad 28: Net-(J5-Pad28) -> GND
- J5 pad 29: Net-(J5-Pad29) -> A13
- J5 pad 3: Net-(J5-Pad3) -> +12VDOWNSTREAM
- J5 pad 30: Net-(J5-Pad30) -> A14
- J5 pad 31: Net-(J5-Pad31) -> A15
- J5 pad 32: Net-(J5-Pad32) -> A16
- J5 pad 33: Net-(J5-Pad33) -> A18
- J5 pad 34: Net-(J5-Pad34) -> A17
- J5 pad 35: Net-(J5-Pad35) -> A20
- J5 pad 36: Net-(J5-Pad36) -> A19
- J5 pad 39: Net-(J5-Pad39) -> GND
- J5 pad 4: Net-(J5-Pad4) -> +12VDOWNSTREAM
- J5 pad 40: Net-(J5-Pad40) -> GND
- J5 pad 5: Net-(J5-Pad5) -> GND
- J5 pad 6: Net-(J5-Pad6) -> GND
- J5 pad 7: Net-(J5-Pad7) -> -12VDOWNSTREAM
- J5 pad 8: Net-(J5-Pad8) -> -12VDOWNSTREAM
- J5 pad 9: Net-(J5-Pad9) -> GND
- J6 pad 1: Net-(J6-Pad1) -> GND
- J6 pad 10: Net-(J6-Pad10) -> /AUDIO_IN_1A
- J6 pad 11: Net-(J6-Pad11) -> /AUDIO_IN_1C
- J6 pad 12: Net-(J6-Pad12) -> /AUDIO_IN_1D
- J6 pad 13: Net-(J6-Pad13) -> GND
- J6 pad 14: Net-(J6-Pad14) -> GND
- J6 pad 15: Net-(J6-Pad15) -> /OSC_D
- J6 pad 16: Net-(J6-Pad16) -> /OSC_C
- J6 pad 17: Net-(J6-Pad17) -> /OSC_B
- J6 pad 18: Net-(J6-Pad18) -> /OSC_A
- J6 pad 19: Net-(J6-Pad19) -> GND
- J6 pad 2: Net-(J6-Pad2) -> GND
- J6 pad 20: Net-(J6-Pad20) -> GND
- J6 pad 21: Net-(J6-Pad21) -> /DAC_2B
- J6 pad 22: Net-(J6-Pad22) -> /DAC_2A
- J6 pad 23: Net-(J6-Pad23) -> /DAC_2C
- J6 pad 24: Net-(J6-Pad24) -> /DAC_2D
- J6 pad 25: Net-(J6-Pad25) -> /DAC_1B
- J6 pad 26: Net-(J6-Pad26) -> /DAC_1A
- J6 pad 27: Net-(J6-Pad27) -> /DAC_1C
- J6 pad 28: Net-(J6-Pad28) -> /DAC_1D
- J6 pad 29: Net-(J6-Pad29) -> GND
- J6 pad 3: Net-(J6-Pad3) -> /AUDIO_OUT_L
- J6 pad 30: Net-(J6-Pad30) -> GND
- J6 pad 31: Net-(J6-Pad31) -> /DAC_4B
- J6 pad 32: Net-(J6-Pad32) -> /DAC_4A
- J6 pad 33: Net-(J6-Pad33) -> /DAC_4C
- J6 pad 34: Net-(J6-Pad34) -> /DAC_4D
- J6 pad 35: Net-(J6-Pad35) -> /DAC_3B
- J6 pad 36: Net-(J6-Pad36) -> /DAC_3A
- J6 pad 37: Net-(J6-Pad37) -> /DAC_3C
- J6 pad 38: Net-(J6-Pad38) -> /DAC_3D
- J6 pad 39: Net-(J6-Pad39) -> GND
- J6 pad 4: Net-(J6-Pad4) -> /AUDIO_OUT_R
- J6 pad 40: Net-(J6-Pad40) -> GND
- J6 pad 5: Net-(J6-Pad5) -> /AUDIO_IN_2B
- J6 pad 6: Net-(J6-Pad6) -> /AUDIO_IN_2A
- J6 pad 7: Net-(J6-Pad7) -> /AUDIO_IN_2C
- J6 pad 8: Net-(J6-Pad8) -> /AUDIO_IN_2D
- J6 pad 9: Net-(J6-Pad9) -> /AUDIO_IN_1B
- J7 pad 1: Net-(J7-Pad1) -> GND
- J7 pad 10: Net-(J7-Pad10) -> GND
- J7 pad 11: Net-(J7-Pad11) -> SERIAL4.0
- J7 pad 12: Net-(J7-Pad12) -> GND
- J7 pad 13: Net-(J7-Pad13) -> SERIAL4.1
- J7 pad 14: Net-(J7-Pad14) -> GND
- J7 pad 15: Net-(J7-Pad15) -> SERIAL4.2
- J7 pad 16: Net-(J7-Pad16) -> GND
- J7 pad 17: Net-(J7-Pad17) -> SERIAL4.3
- J7 pad 18: Net-(J7-Pad18) -> GND
- J7 pad 19: Net-(J7-Pad19) -> DB0
- J7 pad 2: Net-(J7-Pad2) -> GND
- J7 pad 20: Net-(J7-Pad20) -> GND
- J7 pad 21: Net-(J7-Pad21) -> GND
- J7 pad 22: Net-(J7-Pad22) -> GND
- J7 pad 23: Net-(J7-Pad23) -> SERIAL1.0
- J7 pad 24: Net-(J7-Pad24) -> GND
- J7 pad 25: Net-(J7-Pad25) -> SERIAL1.1
- J7 pad 26: Net-(J7-Pad26) -> GND
- J7 pad 27: Net-(J7-Pad27) -> SERIAL1.2
- J7 pad 28: Net-(J7-Pad28) -> GND
- J7 pad 29: Net-(J7-Pad29) -> SERIAL1.3
- J7 pad 3: Net-(J7-Pad3) -> GND
- J7 pad 30: Net-(J7-Pad30) -> GND
- J7 pad 31: Net-(J7-Pad31) -> DR4
- J7 pad 32: Net-(J7-Pad32) -> GND
- J7 pad 33: Net-(J7-Pad33) -> DR3
- J7 pad 34: Net-(J7-Pad34) -> GND
- J7 pad 35: Net-(J7-Pad35) -> DR2
- J7 pad 36: Net-(J7-Pad36) -> GND
- J7 pad 37: Net-(J7-Pad37) -> DR1
- J7 pad 38: Net-(J7-Pad38) -> GND
- J7 pad 39: Net-(J7-Pad39) -> GND
- J7 pad 4: Net-(J7-Pad4) -> GND
- J7 pad 40: Net-(J7-Pad40) -> GND
- J7 pad 5: Net-(J7-Pad5) -> GND
- J7 pad 6: Net-(J7-Pad6) -> GND
- J7 pad 7: Net-(J7-Pad7) -> DB1
- J7 pad 8: Net-(J7-Pad8) -> GND
- J7 pad 9: Net-(J7-Pad9) -> DB2
- R15 pad 1: /Switching/DAC_1 -> /Switching/DAC_3
- R16 pad 1: /Switching/DAC_1 -> /Switching/DAC_4
- R17 pad 1: /Switching/DAC_3 -> /Switching/DAC_1
- R18 pad 1: /Switching/DAC_4 -> /Switching/DAC_2
- R19 pad 1: /Switching/DAC_1 -> /Switching/DAC_3
- R20 pad 1: /Switching/DAC_1 -> /Switching/DAC_4
- R21 pad 1: /Switching/DAC_3 -> /Switching/DAC_1
- R22 pad 1: /Switching/DAC_4 -> /Switching/DAC_2
- R23 pad 1: Net-(R23-Pad1) -> Net-(C21-Pad1)
- R23 pad 2: /Switching/ADC_1 -> A1-PRE
- R24 pad 1: Net-(R23-Pad1) -> Net-(C21-Pad1)
- R25 pad 1: Net-(R25-Pad1) -> Net-(C22-Pad1)
- R25 pad 2: /Switching/ADC_2 -> A2-PRE
- R26 pad 1: Net-(R25-Pad1) -> Net-(C22-Pad1)
- R27 pad 1: Net-(R27-Pad1) -> Net-(C23-Pad1)
- R27 pad 2: /AnalogInBuffers/ANALOG_IN_3 -> A3-PRE
- R28 pad 1: Net-(R27-Pad1) -> Net-(C23-Pad1)
- R29 pad 1: Net-(R29-Pad1) -> Net-(C24-Pad1)
- R29 pad 2: /AnalogInBuffers/ANALOG_IN_4 -> A4-PRE
- R3 pad 2: Net-(C5-Pad2) -> -10V
- R30 pad 1: Net-(R29-Pad1) -> Net-(C24-Pad1)
- R31 pad 1: /AnalogInBuffers/ADC_1 -> A1
- R31 pad 2: Net-(R23-Pad1) -> Net-(C21-Pad1)
- R32 pad 1: /AnalogInBuffers/ADC_2 -> A2
- R32 pad 2: Net-(R25-Pad1) -> Net-(C22-Pad1)
- R33 pad 1: /AnalogInBuffers/ADC_3 -> A3
- R33 pad 2: Net-(R27-Pad1) -> Net-(C23-Pad1)
- R34 pad 1: /AnalogInBuffers/ADC_4 -> A4
- R34 pad 2: Net-(R29-Pad1) -> Net-(C24-Pad1)
- R35 pad 1: Net-(C19-Pad1) -> Net-(C25-Pad1)
- R35 pad 2: GND -> A5-PRE
- R36 pad 1: Net-(C20-Pad1) -> Net-(C25-Pad1)
- R36 pad 2: GND -> -10V
- R37 pad 1: /Switching/AUDIO_IN_1 -> Net-(C26-Pad1)
- R37 pad 2: Net-(C21-Pad1) -> A6-PRE
- R38 pad 1: /Switching/AUDIO_IN_2 -> Net-(C26-Pad1)
- R38 pad 2: Net-(C22-Pad1) -> -10V
- R39 pad 1: /CODEC/L_OUT -> Net-(C27-Pad1)
- R39 pad 2: Net-(C19-Pad1) -> A7-PRE
- R40 pad 1: /CODEC/R_OUT -> Net-(C27-Pad1)
- R40 pad 2: Net-(C20-Pad1) -> -10V
- U1 pad 5: CURRENT_SCL -> I2C_SCL
- U1 pad 6: CURRENT_SDA -> I2C_SDA
- U10 pad 11: (no net) -> -12V
- U10 pad 4: (no net) -> +12V
- U11 pad 1: /AnalogInBuffers/ADC_1 -> A1
- U11 pad 10: Net-(U11-Pad10) -> GND
- U11 pad 11: (no net) -> GND
- U11 pad 12: Net-(U11-Pad12) -> GND
- U11 pad 13: Net-(R29-Pad1) -> Net-(C24-Pad1)
- U11 pad 14: /AnalogInBuffers/ADC_4 -> A4
- U11 pad 2: Net-(R23-Pad1) -> Net-(C21-Pad1)
- U11 pad 3: Net-(U11-Pad3) -> GND
- U11 pad 4: (no net) -> +3V3
- U11 pad 5: Net-(U11-Pad5) -> GND
- U11 pad 6: Net-(R25-Pad1) -> Net-(C22-Pad1)
- U11 pad 7: /AnalogInBuffers/ADC_2 -> A2
- U11 pad 8: /AnalogInBuffers/ADC_3 -> A3
- U11 pad 9: Net-(R27-Pad1) -> Net-(C23-Pad1)
- U12 pad 1: Net-(JP3-Pad2) -> A5
- U12 pad 10: /MCU/I2S_IN_SD -> GND
- U12 pad 11: Net-(C19-Pad2) -> GND
- U12 pad 12: Net-(C20-Pad2) -> GND
- U12 pad 14: GND -> A8
- U12 pad 2: /CODEC/XTO -> Net-(C25-Pad1)
- U12 pad 4: Net-(FB5-Pad1) -> +3V3
- U12 pad 5: Net-(U12-Pad5) -> GND
- U12 pad 6: /CODEC/I2S_SCK -> Net-(C26-Pad1)
- U12 pad 7: /CODEC/I2S_OUT_SD -> A6
- U12 pad 8: /CODEC/I2S_OUT_WS -> A7
- U12 pad 9: /CODEC/I2S_IN_SD -> Net-(C27-Pad1)
- U2 pad 5: CURRENT_SCL -> I2C_SCL
- U2 pad 6: CURRENT_SDA -> I2C_SDA
- U4 pad 2: Net-(C5-Pad2) -> -10V
- U5 pad 10: Net-(U5-Pad10) -> A10
- U5 pad 11: Net-(U5-Pad11) -> A11
- U5 pad 12: Net-(U5-Pad12) -> A12
- U5 pad 13: Net-(U5-Pad13) -> A13
- U5 pad 14: Net-(U5-Pad14) -> A14
- U5 pad 15: Net-(U5-Pad15) -> A15
- U5 pad 16: Net-(U5-Pad16) -> A16
- U5 pad 17: /CODEC/I2S_MCLK -> A18
- U5 pad 18: /CODEC/I2S_OUT_WS -> A17
- U5 pad 19: /CODEC/I2S_SCK -> A20
- U5 pad 20: /CODEC/I2S_OUT_SD -> A19
- U5 pad 23: /MCU/I2S_IN_SD -> DB1
- U5 pad 24: /MCU/I2S_FS1 -> DB2
- U5 pad 25: /MCU/I2S_SCK1 -> SERIAL4.0
- U5 pad 26: /MCU/I2S_MCK1 -> SERIAL4.1
- U5 pad 27: Net-(U5-Pad27) -> SERIAL4.2
- U5 pad 28: Net-(U5-Pad28) -> SERIAL4.3
- U5 pad 29: Net-(U5-Pad29) -> DB0
- U5 pad 3: Net-(U5-Pad3) -> A5
- U5 pad 30: Net-(U5-Pad30) -> SPI_SCLK
- U5 pad 31: Net-(U5-Pad31) -> /MCU/DAC_CS
- U5 pad 32: Net-(U5-Pad32) -> SPI_COPI
- U5 pad 35: Net-(U5-Pad35) -> SERIAL1.0
- U5 pad 36: Net-(U5-Pad36) -> SERIAL1.1
- U5 pad 37: Net-(U5-Pad37) -> SERIAL1.2
- U5 pad 38: Net-(U5-Pad38) -> SERIAL1.3
- U5 pad 39: Net-(U5-Pad39) -> DR4
- U5 pad 4: Net-(U5-Pad4) -> A6
- U5 pad 40: Net-(U5-Pad40) -> DR3
- U5 pad 41: Net-(U5-Pad41) -> DR2
- U5 pad 42: Net-(U5-Pad42) -> DR1
- U5 pad 43: Net-(U5-Pad43) -> /MCU/DOTSTAR_DI
- U5 pad 44: Net-(U5-Pad44) -> /MCU/DOTSTAR_CI
- U5 pad 5: Net-(U5-Pad5) -> A7
- U5 pad 52: Net-(U5-Pad52) -> /MCU/RESET
- U5 pad 59: Net-(U5-Pad59) -> I2C_SDA
- U5 pad 6: Net-(U5-Pad6) -> A8
- U5 pad 60: Net-(U5-Pad60) -> I2C_SCL
- U5 pad 61: Net-(U5-Pad61) -> A1
- U5 pad 62: Net-(U5-Pad62) -> A2
- U5 pad 63: Net-(U5-Pad63) -> A3
- U5 pad 64: Net-(U5-Pad64) -> A4
- U5 pad 9: Net-(U5-Pad9) -> A9
- U6 pad 12: /MCU/DAC_SCLK -> SPI_SCLK
- U6 pad 14: /MCU/DAC_SDIN -> SPI_COPI
- U6 pad 5: Net-(FB4-Pad2) -> Net-(C16-Pad1)
- U7 pad 1: /Switching/SCK -> SPI_SCLK
- U7 pad 10: /Switching/AUDIO_IN_1C -> /AUDIO_IN_1C
- U7 pad 11: /Switching/AUDIO_IN_1 -> /AUDIO_IN_L
- U7 pad 12: /Switching/AUDIO_IN_1D -> /AUDIO_IN_1D
- U7 pad 13: /Switching/AUDIO_IN_2A -> /AUDIO_IN_2A
- U7 pad 14: /Switching/AUDIO_IN_2 -> /AUDIO_IN_R
- U7 pad 15: /Switching/AUDIO_IN_2B -> /AUDIO_IN_2B
- U7 pad 16: /Switching/AUDIO_IN_2 -> /AUDIO_IN_R
- U7 pad 17: /Switching/AUDIO_IN_2C -> /AUDIO_IN_2C
- U7 pad 18: /Switching/AUDIO_IN_2 -> /AUDIO_IN_R
- U7 pad 19: /Switching/AUDIO_IN_2D -> /AUDIO_IN_2D
- U7 pad 20: /Switching/AUDIO_IN_2 -> /AUDIO_IN_R
- U7 pad 3: /Switching/SDI -> SPI_COPI
- U7 pad 5: /Switching/AUDIO_IN_1 -> /AUDIO_IN_L
- U7 pad 6: /Switching/AUDIO_IN_1A -> /AUDIO_IN_1A
- U7 pad 7: /Switching/AUDIO_IN_1 -> /AUDIO_IN_L
- U7 pad 8: /Switching/AUDIO_IN_1B -> /AUDIO_IN_1B
- U7 pad 9: /Switching/AUDIO_IN_1 -> /AUDIO_IN_L
- U8 pad 1: /Switching/SCK -> SPI_SCLK
- U8 pad 10: /Switching/DAC_2A -> /DAC_1C
- U8 pad 12: /Switching/DAC_2B -> /DAC_1D
- U8 pad 13: /Switching/DAC_3A -> /DAC_2A
- U8 pad 14: /Switching/DAC_3 -> /Switching/DAC_2
- U8 pad 15: /Switching/DAC_3B -> /DAC_2B
- U8 pad 16: /Switching/DAC_3 -> /Switching/DAC_2
- U8 pad 17: /Switching/DAC_4A -> /DAC_2C
- U8 pad 18: /Switching/DAC_4 -> /Switching/DAC_2
- U8 pad 19: /Switching/DAC_4B -> /DAC_2D
- U8 pad 20: /Switching/DAC_4 -> /Switching/DAC_2
- U8 pad 6: /Switching/DAC_1A -> /DAC_1A
- U8 pad 8: /Switching/DAC_1B -> /DAC_1B
- U9 pad 1: /Switching/SCK -> SPI_SCLK
- U9 pad 10: /Switching/ADC_1C -> /DAC_3C
- U9 pad 11: /Switching/ADC_1 -> /Switching/DAC_3
- U9 pad 12: /Switching/ADC_1D -> /DAC_3D
- U9 pad 13: /Switching/ADC_2A -> /DAC_4A
- U9 pad 14: /Switching/ADC_2 -> /Switching/DAC_4
- U9 pad 15: /Switching/ADC_2B -> /DAC_4B
- U9 pad 16: /Switching/ADC_2 -> /Switching/DAC_4
- U9 pad 17: /Switching/ADC_2C -> /DAC_4C
- U9 pad 18: /Switching/ADC_2 -> /Switching/DAC_4
- U9 pad 19: /Switching/ADC_2D -> /DAC_4D
- U9 pad 20: /Switching/ADC_2 -> /Switching/DAC_4
- U9 pad 5: /Switching/ADC_1 -> /Switching/DAC_3
- U9 pad 6: /Switching/ADC_1A -> /DAC_3A
- U9 pad 7: /Switching/ADC_1 -> /Switching/DAC_3
- U9 pad 8: /Switching/ADC_1B -> /DAC_3B
- U9 pad 9: /Switching/ADC_1 -> /Switching/DAC_3
Routing:
- net +3V3: track 0.00 -> 348.1 mm, vias 0 -> 14
- net -10V: track 0.00 -> 208.9 mm, vias 0 -> 9
- net -12V: track 0.00 -> 139.0 mm, vias 0 -> 6
- net +12V: track 0.00 -> 129.0 mm, vias 0 -> 6
- net D+: track 0.00 -> 96.7 mm
- net D-: track 0.00 -> 95.6 mm
- net SPI_SCLK: track 0.00 -> 90.9 mm, vias 0 -> 4
- net /OSC_A: track 0.00 -> 86.7 mm
- net /OSC_B: track 0.00 -> 79.1 mm
- net /OSC_C: track 0.00 -> 65.5 mm
- net A19: track 0.00 -> 60.3 mm
- net A14: track 0.00 -> 59.8 mm
- net A17: track 0.00 -> 59.5 mm
- net /OSC_D: track 0.00 -> 59.0 mm
- net A16: track 0.00 -> 58.8 mm
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- added copper zone on B.Cu, net GND
- added copper zone on F.Cu, net GND
Other:
- net class 12V added: clearance 0.3, trace_width 0.4, via_dia 0.8, via_drill 0.5
- net class 3.3V added: clearance 0.2, trace_width 0.25, via_dia 0.7, via_drill 0.3
- net class Absolute minimum added: clearance 0.15, trace_width 0.15, via_dia 0.7, via_drill 0.3
- net class Analog added: clearance 0.2, trace_width 0.2, via_dia 0.7, via_drill 0.3
- net class Default: clearance 0.2 -> 0.17; trace_width 0.25 -> 0.16; via_dia 0.8 -> 0.7; via_drill 0.4 -> 0.3
- rule pad_to_mask_clearance: 0.05 -> 0.0508
- rule trace_clearance: 0.2 -> 0.17
- rule trace_min: 0.2 -> 0.15
- rule via_min_size: 0.4 -> 0.5
- board text added: "*"
