File: hardware/board/AnalogInBuffers.sch (KiCad schematic (older format))
At the start: 54 parts, among them U11 MCP6004, U12 MCP6004, U13 MCP6004

Commit message: Re-do the motherboard
Parts:
- removed C20: 0.1uF, Capacitor_SMD:C_0603_1608Metric_Pad1.08x0.95mm_HandSolder, symbol Device:C_Small
- removed C25, C26, C27, C28, C29, C30, C31, C32: 22pF, Capacitor_SMD:C_0603_1608Metric_Pad1.08x0.95mm_HandSolder, symbol Device:C_Small
- removed R35, R39, R41, R47, R49, R51, R53: 100k, Resistor_SMD:R_0603_1608Metric_Pad0.98x0.95mm_HandSolder, symbol Device:R_US
- removed R36, R38, R40, R42, R48, R50, R52, R54: 121k, Resistor_SMD:R_0603_1608Metric_Pad0.98x0.95mm_HandSolder, symbol Device:R_US
- removed R43, R44, R45, R46, R55, R56, R57, R58: 18.7k, Resistor_SMD:R_0603_1608Metric_Pad0.98x0.95mm_HandSolder, symbol Device:R_US
- removed U12, U13: MCP6004, Package_SO:TSSOP-14_4.4x5mm_P0.65mm, symbol winterbloom:MCP6004
- added U3: LM4040-10, Package_TO_SOT_SMD:SOT-23, symbol winterbloom:LM4040-10
- R37: value 100k -> 1k
- renumbered C18 to C20
Connections:
- net A6-PRE is gone; now on net -10v_ADC: R37.2
- net +3V3: no longer C19.1
- net GND: now also C19.1, U3.1 (K); no longer C19.2
- net -12V: now reaches R37.1
- net -10V renamed -10v_ADC
- net -10v_ADC: now also C19.2, U3.2 (A)
- net A1 renamed ADC_1_POST
- net A1-PRE renamed ADC_1_PRE
- net A2 renamed ADC_2_POST
- net A2-PRE renamed ADC_2_PRE
- net A3 renamed ADC_3_POST
- net A3-PRE renamed ADC_3_PRE
- net A4 renamed ADC_4_POST
- net A4-PRE renamed ADC_4_PRE
Other:
- moved on the sheet: C20, U11E
