File: hardware/board/switching.sch (KiCad schematic (older format))
At the start: 5 parts, among them U7 ADG1414BRU, U8 ADG1414BRU, U9 ADG1414BRU

Commit message: Re-do the motherboard
Parts:
- removed R5, R6: 1k, Resistor_SMD:R_0603_1608Metric_Pad0.98x0.95mm_HandSolder, symbol Device:R_US
- removed U7, U8, U9: ADG1414BRU, Package_SO:TSSOP-24_4.4x7.8mm_P0.65mm, symbol Analog_Switch:ADG1414BRU
- added C25, C26, C27, C28, C29, C30, C31, C32: 0.1uF, Capacitor_SMD:C_0603_1608Metric_Pad1.08x0.95mm_HandSolder, symbol Device:C_Small
- added U4, U7, U8, U9: MUX509, Package_SO:TSSOP-16_4.4x5mm_P0.65mm, symbol winterbloom:MUX509
Connections:
- net +12V: now also C29.1, C30.1, C31.1, C32.1, U4.14 (VDD), U4.2 (EN), U7.14 (VDD), U7.2 (EN), U8.14 (VDD), U8.2 (EN), U9.14 (VDD), U9.2 (EN)
- net -12V: now also C25.1, C26.1, C27.1, C28.1, U4.3 (VSS), U7.3 (VSS), U8.3 (VSS), U9.3 (VSS)
- net DAC_1: now also U9.8 (DA)
- net DAC_1A: now also U9.4 (S1A)
- net DAC_1B: now also U9.5 (S2A)
- net DAC_1C: now also U9.6 (S3A)
- net DAC_1D: now also U9.7 (S4A)
- net DAC_2: now also U4.9 (DB)
- net DAC_2A: now also U4.13 (S1B)
- net DAC_2B: now also U4.12 (S2B)
- net DAC_2C: now also U4.11 (S3B)
- net DAC_2D: now also U4.10 (S4B)
- net DAC_3: now also U4.8 (DA)
- net DAC_3A: now also U4.4 (S1A)
- net DAC_3B: now also U4.5 (S2A)
- net DAC_3C: now also U4.6 (S3A)
- net DAC_3D: now also U4.7 (S4A)
- net DAC_4: now also U9.9 (DB)
- net DAC_4A: now also U9.13 (S1B)
- net DAC_4B: now also U9.12 (S2B)
- net DAC_4C: now also U9.11 (S3B)
- net DAC_4D: now also U9.10 (S4B)
- net GND: now also C25.2, C26.2, C27.2, C28.2, C29.2, C30.2, C31.2, C32.2, U4.15 (GND), U7.15 (GND), U8.15 (GND), U9.15 (GND)
- new net ADC_1: U7.8 (DA)
- new net ADC_1A: U7.4 (S1A)
- new net ADC_1B: U7.5 (S2A)
- new net ADC_1C: U7.6 (S3A)
- new net ADC_1D: U7.7 (S4A)
- new net ADC_2: U8.9 (DB)
- new net ADC_2A: U8.13 (S1B)
- new net ADC_2B: U8.12 (S2B)
- new net ADC_2C: U8.11 (S3B)
- new net ADC_2D: U8.10 (S4B)
- new net ADC_3: U8.8 (DA)
- new net ADC_3A: U8.4 (S1A)
- new net ADC_3B: U8.5 (S2A)
- new net ADC_3C: U8.6 (S3A)
- new net ADC_3D: U8.7 (S4A)
- new net ADC_4: U7.9 (DB)
- new net ADC_4A: U7.13 (S1B)
- new net ADC_4B: U7.12 (S2B)
- new net ADC_4C: U7.11 (S3B)
- new net ADC_4D: U7.10 (S4B)
- new net ADC_A0: U7.1 (A0), U8.1 (A0)
- new net ADC_A1: U7.16 (A1), U8.16 (A1)
- new net DAC_A0: U4.1 (A0), U9.1 (A0)
- new net DAC_A1: U4.16 (A1), U9.16 (A1)
- no-connect marks 1 -> 0
Other:
- note removed: "Analog in 2:8 multiplexer"
- note removed: "Analog out 2:8 multiplexer"
- note removed: "Audio in 8:2 multiplexer"
- note removed: "bypass caps?"
