File: hardware/board/hubble.kicad_pcb (KiCad board)
At the start: 2 copper layers, 100 x 100 mm, 125 parts, among them J1 POWER, J10 Dotstars, J11 USB, J12 FRONT, J2 SWD, J3 USB B, J4 EXT, J5 Left, J6 Right, J7 Bottom, J8 EXT, J9 EXT, SW1 POWER, SW2 Reset, U1 LD1117-3.3, U10 OPA4197, U11 MCP6004, U2 LM4040-10, U3 LM4040-10, U4 MUX509, U5 ATSAMD51J20A-M, U6 AD5689R?RUZ, U7 MUX509, U8 MUX509, U9 MUX509, Y1 32.768 kHz

Commit message: Update design files to KiCAD 6
Other:
- net class 12V removed
- net class 3.3V removed
- net class Absolute minimum removed
- net class Analog removed
- net class Default removed
