File: hardware/board/hubble.kicad_sch (KiCad schematic)
At the start: 7 parts, among them J12 FRONT, J4 EXT, J5 Left, J6 Right, J7 Bottom, J8 EXT, J9 EXT

Commit message: Initial stab at hardware revision
Parts:
- removed J12: FRONT, Connector_PinHeader_2.54mm:PinHeader_2x04_P2.54mm_Vertical, symbol Connector_Generic:Conn_02x04_Odd_Even
- removed J4, J8, J9: EXT, Connector_Wire:SolderWire-0.75sqmm_1x06_P4.8mm_D1.25mm_OD2.3mm, symbol Connector_Generic:Conn_01x06
- removed J5: Left, Connector_PinSocket_2.54mm:PinSocket_2x20_P2.54mm_Vertical, symbol Connector_Generic:Conn_02x20_Odd_Even
- removed J6: Right, Connector_PinSocket_2.54mm:PinSocket_2x20_P2.54mm_Vertical, symbol Connector_Generic:Conn_02x20_Odd_Even
- removed J7: Bottom, Connector_PinSocket_2.54mm:PinSocket_2x20_P2.54mm_Vertical, symbol Connector_Generic:Conn_02x20_Odd_Even
Connections:
- no-connect marks 0 -> 1
Other:
- removed sheet AnalogInBuffers
- removed sheet AnalogOutBuffers
- removed sheet DAC
- removed sheet Switching
- added sheet Analog Ins 1-4 (analog-ins.kicad_sch)
- added sheet Analog Ins 5-8 (analog-ins.kicad_sch)
- added sheet Analog Ins 9-12 (analog-ins.kicad_sch)
- added sheet Analog Outs 1-4 (analog-outs.kicad_sch)
- added sheet Analog Outs 5-8 (analog-outs.kicad_sch)
- added sheet Analog Outs 9-12 (analog-outs.kicad_sch)
- added sheet External IO (external-io.kicad_sch)
- added sheet Low Voltage Analog Ins 13-16 (analog-ins-low-voltage.kicad_sch)
- added sheet Low Voltage Analog Outs 13-16 (analog-outs-low-voltage.kicad_sch)
- added sheet MCU IO (mcu-io.kicad_sch)
- sheet MCU ports: added AIN1, AIN10, AIN11, AIN12, AIN13, AIN14, AIN15, AIN16, AIN2, AIN3, AIN4, AIN5, AIN6, AIN7, AIN8, AIN9, DAC_SCK, DAC_SDO, DOTSTAR_SCK, DOTSTAR_SDO, DS_POWER_EN, GPIO1, GPIO10, GPIO11, GPIO12, GPIO13, GPIO14, GPIO15, GPIO16, GPIO17, GPIO18, GPIO19, GPIO2, GPIO20, GPIO21, GPIO22, GPIO23, GPIO24, GPIO25, GPIO26, GPIO27, GPIO28, GPIO29, GPIO3, GPIO30, GPIO4, GPIO5, GPIO6, GPIO7, GPIO8, GPIO9, QWIIC_SCL, QWIIC_SDA, SDO, SERIAL1.0, SERIAL1.1, SERIAL1.2, SERIAL1.3, SERIAL2.0, SERIAL2.1, SERIAL2.2, SERIAL2.3, SWCLK, SWDIO, USB_D+, USB_D-, ~{RESET}; removed A1, A2, A3, A4, PA02+DAC0, PA04, PA05+DAC1, PA06, PA07, PA08, PA09, PA10, PA11, PA12, PA20, PA21, PA27, PB00, PB01, PB02, PB03, PB06, PB07, PB10, PB11, PB16, PB17, PB22, PB23, PB30, PB31, SPI_COPI, SPI_SCK
- sheet Power ports: added DS_POWER_EN; removed none
